Commit message: new urdf

File: urdf/robot_esr_v2_rev.urdf (robot description, URDF)
Before this commit: robot robot_esr_v2_rev, 35 links, 34 joints
Links:
- link base_link: geometry collision mesh filename=package://robot_esr_v2_rev/meshes/base_link.STL; visual mesh filename=/home/grace/hvac/meshes/base_link.STL

Commit message: ipdate urdf path

File: urdf/robot_esr_v2_rev.urdf (robot description, URDF)
Before this commit: robot robot_esr_v2_rev, 35 links, 34 joints
Links:
- link base_link: geometry collision mesh filename=../meshes/base_link.STL; visual mesh filename=../meshes/base_link.STL
- link body_pitch: geometry collision mesh filename=../meshes/body_pitch.STL; visual mesh filename=../meshes/body_pitch.STL
- link body_yaw: geometry collision mesh filename=../meshes/body_yaw.STL; visual mesh filename=../meshes/body_yaw.STL
- link head_pitch: geometry collision mesh filename=../meshes/head_pitch.STL; visual mesh filename=../meshes/head_pitch.STL
- link head_yaw: geometry collision mesh filename=../meshes/head_yaw.STL; visual mesh filename=../meshes/head_yaw.STL
- link left_arm_pitch_1: geometry collision mesh filename=../meshes/left_arm_pitch_1.STL; visual mesh filename=../meshes/left_arm_pitch_1.STL
- link left_arm_roll_1: geometry collision mesh filename=../meshes/left_arm_roll_1.STL; visual mesh filename=../meshes/left_arm_roll_1.STL
- link left_arm_roll_3: geometry collision mesh filename=../meshes/left_arm_roll_3.STL; visual mesh filename=../meshes/left_arm_roll_3.STL
- link left_arm_roll_5: geometry collision mesh filename=../meshes/left_arm_roll_5.STL; visual mesh filename=../meshes/left_arm_roll_5.STL
- link left_arm_yaw_1: geometry collision mesh filename=../meshes/left_arm_yaw_1.STL; visual mesh filename=../meshes/left_arm_yaw_1.STL
- link left_finger_1: geometry collision mesh filename=../meshes/left_finger_1.STL; visual mesh filename=../meshes/left_finger_1.STL
- link left_finger_3: geometry collision mesh filename=../meshes/left_finger_3.STL; visual mesh filename=../meshes/left_finger_3.STL
- link left_knee_pitch_1: geometry collision mesh filename=../meshes/left_knee_pitch_1.STL; visual mesh filename=../meshes/left_knee_pitch_1.STL
- link left_knee_pitch_3: geometry collision mesh filename=../meshes/left_knee_pitch_3.STL; visual mesh filename=../meshes/left_knee_pitch_3.STL
- link left_knee_pitch_5: geometry collision mesh filename=../meshes/left_knee_pitch_5.STL; visual mesh filename=../meshes/left_knee_pitch_5.STL
- link left_knee_roll_1: geometry collision mesh filename=../meshes/left_knee_roll_1.STL; visual mesh filename=../meshes/left_knee_roll_1.STL
- link left_knee_roll_5: geometry collision mesh filename=../meshes/left_knee_roll_5.STL; visual mesh filename=../meshes/left_knee_roll_5.STL
- link left_knee_yaw_1: geometry collision mesh filename=../meshes/left_knee_yaw_1.STL; visual mesh filename=../meshes/left_knee_yaw_1.STL
- link left_thumb_1: geometry collision mesh filename=../meshes/left_thumb_1.STL; visual mesh filename=../meshes/left_thumb_1.STL
- link left_thumb_3: geometry collision mesh filename=../meshes/left_thumb_3.STL; visual mesh filename=../meshes/left_thumb_3.STL
- link right_arm_pitch_2: geometry collision mesh filename=../meshes/right_arm_pitch_2.STL; visual mesh filename=../meshes/right_arm_pitch_2.STL
- link right_arm_roll_2: geometry collision mesh filename=../meshes/right_arm_roll_2.STL; visual mesh filename=../meshes/right_arm_roll_2.STL
- link right_arm_roll_4: geometry collision mesh filename=../meshes/right_arm_roll_4.STL; visual mesh filename=../meshes/right_arm_roll_4.STL
- link right_arm_roll_6: geometry collision mesh filename=../meshes/right_arm_roll_6.STL; visual mesh filename=../meshes/right_arm_roll_6.STL
- link right_arm_yaw_2: geometry collision mesh filename=../meshes/right_arm_yaw_2.STL; visual mesh filename=../meshes/right_arm_yaw_2.STL
- link right_finger_2: geometry collision mesh filename=../meshes/right_finger_2.STL; visual mesh filename=../meshes/right_finger_2.STL
- link right_finger_4: geometry collision mesh filename=../meshes/right_finger_4.STL; visual mesh filename=../meshes/right_finger_4.STL
- link right_knee_pitch_2: geometry collision mesh filename=../meshes/right_knee_pitch_2.STL; visual mesh filename=../meshes/right_knee_pitch_2.STL
- link right_knee_pitch_4: geometry collision mesh filename=../meshes/right_knee_pitch_4.STL; visual mesh filename=../meshes/right_knee_pitch_4.STL
- link right_knee_pitch_6: geometry collision mesh filename=../meshes/right_knee_pitch_6.STL; visual mesh filename=../meshes/right_knee_pitch_6.STL
- link right_knee_roll_2: geometry collision mesh filename=../meshes/right_knee_roll_2.STL; visual mesh filename=../meshes/right_knee_roll_2.STL
- link right_knee_roll_6: geometry collision mesh filename=../meshes/right_knee_roll_6.STL; visual mesh filename=../meshes/right_knee_roll_6.STL
- link right_knee_yaw_2: geometry collision mesh filename=../meshes/right_knee_yaw_2.STL; visual mesh filename=../meshes/right_knee_yaw_2.STL
- link right_thumb_2: geometry collision mesh filename=../meshes/right_thumb_2.STL; visual mesh filename=../meshes/right_thumb_2.STL
- link right_thumb_4: geometry collision mesh filename=../meshes/right_thumb_4.STL; visual mesh filename=../meshes/right_thumb_4.STL
