Commit message: nambahin floor

File: urdf/robot_esr_v2_rev.urdf (robot description, URDF)
Before this commit: robot robot_esr_v2_rev, 35 links, 34 joints
Links:
- added link root_x_link
- added link root_y_link
- added link root_yaw_link
- added link root_z_link
- added link world
Joints:
- added joint root_base_fixed_joint: type fixed, parent root_yaw_link, child base_link, origin xyz=0 0 0 rpy=0 0 0
- added joint root_x_joint: type prismatic, parent world, child root_x_link, origin xyz=0 0 0 rpy=0 0 0, axis 1 0 0, limit lower=-100 upper=100 effort=1000 velocity=10
- added joint root_y_joint: type prismatic, parent root_x_link, child root_y_link, origin xyz=0 0 0 rpy=0 0 0, axis 0 1 0, limit lower=-100 upper=100 effort=1000 velocity=10
- added joint root_yaw_joint: type revolute, parent root_z_link, child root_yaw_link, origin xyz=0 0 0 rpy=0 0 0, axis 0 0 1, limit lower=-6.28318 upper=6.28318 effort=1000 velocity=3
- added joint root_z_joint: type prismatic, parent root_y_link, child root_z_link, origin xyz=0 0 0 rpy=0 0 0, axis 0 0 1, limit lower=-100 upper=100 effort=1000 velocity=10
